File: parcialinfo22.brd (EAGLE design)
At the start: 68.6 x 53.3 mm, 137 parts

Commit message: implementacion en tinkercad
Parts:
- removed D1, D2, D3, D4: (no value), AUTODESK_CIRCUITS_BREADBOARD:LED5MM
- added D65, D66, D67, D68: (no value), AUTODESK_CIRCUITS_BREADBOARD:LED5MM
- moved D43 876.3 mm to (5.00, 594.3)
- moved D44 876.3 mm to (5.00, 607.0)
- moved D45 876.3 mm to (5.00, 619.7)
- moved D46 876.3 mm to (5.00, 632.4)
- moved D47 876.3 mm to (5.00, 645.1)
- moved D48 876.3 mm to (5.00, 657.8)
- moved D49 876.3 mm to (5.00, 670.5)
- moved D50 876.3 mm to (5.00, 683.2)
- moved D51 876.3 mm to (5.00, 695.9)
- moved D52 876.3 mm to (5.00, 708.6)
- moved D53 876.3 mm to (5.00, 721.3)
- moved D54 876.3 mm to (5.00, 734.0)
- moved D55 876.3 mm to (5.00, 746.7)
- moved D56 876.3 mm to (5.00, 759.4)
- moved D57 876.3 mm to (5.00, 772.1)
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Connections:
- removed net N$141 (its old number): D61.A, R36.2
- removed net N$97 (its old number): D8.A, R19.2
- new net N$75: D20.A, R58.1
- new net N$76: D19.A, R8.2
- net N$100: now also D35.A, R29.2; no longer D59.A, R22.2
- net N$101: now also D34.A, R28.2; no longer D51.A, R60.1
- net N$102: now also D33.A, R27.2; no longer D9.A, R23.2
- net N$103: now also D32.A, R26.2; no longer D13.A, R24.2
- net N$104: now also D31.A; no longer D21.A
- net N$105: now also D30.A, R24.2; no longer D28.A, R26.2
- net N$106: now also D29.A, R23.2; no longer D36.A, R27.2
- net N$107: now also D36.A, R61.1; no longer D44.A, R28.2
- net N$108: now also D44.A, R62.1; no longer D60.A, R29.2
- net N$109: now also R63.1; no longer R61.1
- net N$110: now also D60.A, R64.1; no longer D5.A, R30.2
- net N$111: now also D68.A, R65.1; no longer D14.A, R31.2
- net N$112: now also D43.A, R36.2; no longer D22.A, R32.2
- net N$113: now also D42.A, R35.2; no longer D29.A, R34.2
- net N$114: now also D41.A; no longer D37.A
- net N$115: now also D40.A, R34.2; no longer D45.A, R35.2
- net N$116: now also D39.A, R32.2; no longer D53.A, R62.1
- net N$117: now also D38.A, R31.2; no longer D6.A, R43.2
- net N$118: now also D37.A, R30.2; no longer D15.A, R42.2
- net N$119: now also D51.A, R37.2; no longer D23.A, R40.2
- net N$120: now also D50.A, R38.2; no longer D30.A, R41.2
- net N$121: now also D49.A; no longer D38.A
- net N$122: now also D48.A, R41.2; no longer D46.A, R38.2
- net N$123: now also D47.A, R40.2; no longer D62.A, R37.2
- net N$124: now also D46.A, R42.2; no longer D54.A, R63.1
- net N$125: now also D45.A, R43.2; no longer D7.A, R49.2
- net N$126: now also D59.A, R44.2; no longer D16.A, R48.2
- net N$127: now also D58.A, R45.2; no longer D1.A, R57.2
- net N$128: now also D57.A, R50.2; no longer D17.A, R56.2
- net N$129: now also D56.A, R46.2; no longer D25.A, R55.2
- net N$130: now also D55.A, R47.2; no longer D32.A, R53.2
- net N$131: now also D54.A, R48.2; no longer D40.A, R54.2
- net N$132: now also D53.A, R49.2; no longer D48.A, R52.2
- net N$133: now also D67.A; no longer D64.A
- net N$134: now also D66.A, R52.2; no longer D56.A, R65.1
- net N$135: now also D65.A, R54.2; no longer D24.A, R47.2
- net N$136: now also D64.A, R53.2; no longer D31.A, R46.2
- net N$137: now also D63.A, R55.2; no longer D39.A, R50.2
- net N$138: now also D62.A, R56.2; no longer D47.A, R45.2
- net N$139: now also D61.A, R57.2; no longer D63.A, R44.2
- net N$140: now also D10.K, D11.K, D12.K, D13.K, D14.K, D15.K, D16.K, D17.K, D18.K, D19.K, D20.K, D21.K, D22.K, D23.K, D24.K, D25.K, D26.K, D27.K, D28.K, D29.K, D30.K, D31.K, D32.K, D33.K, D34.K, D35.K, D36.K, D37.K, D38.K, D39.K, D40.K, D41.K, D42.K, D43.K, D44.K, D45.K, D46.K, D47.K, D48.K, D49.K, D5.K, D50.K, D51.K, D52.K, D53.K, D54.K, D55.K, D56.K, D57.K, D58.K, D59.K, D6.K, D60.K, D61.K, D62.K, D63.K, D64.K, D65.K, D66.K, D67.K, D68.K, D7.K, D8.K, D9.K, U1.GND.., U2.13, U2.8, U3.13, U3.8, U4.13, U4.8, U5.13, U5.8, U6.13, U6.8, U7.13, U7.8, U8.13, U8.8, U9.13, U9.8; no longer D55.A, R64.1
- net N$77: now also D18.A, R7.2; no longer D1.K, D10.K, D11.K, D12.K, D13.K, D14.K, D15.K, D16.K, D17.K, D18.K, D19.K, D2.K, D20.K, D21.K, D22.K, D23.K, D24.K, D25.K, D26.K, D27.K, D28.K, D29.K, D3.K, D30.K, D31.K, D32.K, D33.K, D34.K, D35.K, D36.K, D37.K, D38.K, D39.K, D4.K, D40.K, D41.K, D42.K, D43.K, D44.K, D45.K, D46.K, D47.K, D48.K, D49.K, D5.K, D50.K, D51.K, D52.K, D53.K, D54.K, D55.K, D56.K, D57.K, D58.K, D59.K, D6.K, D60.K, D61.K, D62.K, D63.K, D64.K, D7.K, D8.K, D9.K, U1.GND.., U2.13, U2.8, U3.13, U3.8, U4.13, U4.8, U5.13, U5.8, U6.13, U6.8, U7.13, U7.8, U8.13, U8.8, U9.13, U9.8
- net N$78: now also D17.A, R6.2; no longer D10.A, R3.2
- net N$79: now also D16.A, R5.2; no longer D2.A, R1.2
- net N$80: now also D15.A; no longer D18.A
- net N$81: now also D14.A, R3.2; no longer D26.A, R5.2
- net N$82: now also D13.A, R1.2; no longer D33.A, R6.2
- net N$83: now also D11.A, R15.2; no longer D41.A, R7.2
- net N$84: now also D10.A, R14.2; no longer D57.A, R8.2
- net N$85: now also D9.A, R13.2; no longer D49.A, R58.1
- net N$86: now also D8.A, R12.2; no longer D3.A, R9.2
- net N$87: now also D7.A, R11.2; no longer D11.A, R10.2
- net N$88: now also D6.A, R10.2; no longer D19.A, R11.2
- net N$89: now also D5.A, R9.2; no longer D27.A, R12.2
- net N$90: now also D25.A, R20.2; no longer D34.A, R13.2
- net N$91: now also D26.A, R21.2; no longer D42.A, R14.2
- net N$92: now also D27.A, R22.2; no longer D58.A, R15.2
- net N$93: now also D24.A, R19.2; no longer D50.A, R59.1
- net N$94: now also D23.A, R17.2; no longer D4.A, R16.2
- net N$95: now also D22.A; no longer D12.A
- net N$96: now also D21.A, R16.2; no longer D20.A, R17.2
- net N$98: now also D12.A, R59.1; no longer D35.A, R20.2
- net N$99: now also D28.A, R60.1; no longer D43.A, R21.2
